File: ZYNQ_Pi_Zero.kicad_sch (KiCad schematic)
At the start: 1 part, among them U1 xc7z010clg400

Commit message: feat: finish bank0 & qspi sch design
Parts:
- removed unit 1 of U1
Other:
- added sheet BANK0 (bank0.kicad_sch)

Commit message: feat: finish basic power sch design
Parts:
- removed unit 8 of U1
Other:
- added sheet POWER (power.kicad_sch)

Commit message: feat: finish basic hdmi sch design
Other:
- added sheet HDMI (HDMI.kicad_sch)
Changed lines of the file:
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@@
+		)
+	)
+	(sheet
+		(at 381 127)
+		(size 50.8 38.1)
+		(exclude_from_sim no)
+		(in_bom yes)
+		(on_board yes)
+		(dnp no)
+		(fields_autoplaced yes)
+		(stroke
+			(width 0.1524)
+			(type solid)
+		)
+		(fill
+			(color 0 0 0 0)
+		)
+		(property "Sheetname" "HDMI"
+			(at 381 126.2884 0)
+			(show_name no)
+			(do_not_autoplace no)
+			(effects
+				(font
+					(size 1.27 1.27)
+				)
+				(justify left bottom)
+			)
+		)
+		(property "Sheetfile" "HDMI.kicad_sch"
+			(at 381 165.6846 0)
+			(show_name no)
+			(do_not_autoplace no)
+			(effects
+				(font
+					(size 1.27 1.27)
+				)
+				(justify left top)
+			)
+		)
+		(instances
+			(project "ZYNQ_Pi_Zero"
+				(path "/239d02af-7f9c-469f-b86b-abe2695ec54e"
+					(page "5")
+				)
+			)
 		)
 	)
