File: ZYNQ_Pi_Zero.kicad_sch (KiCad schematic)
At the start: 1 part, among them U101 xc7z010clg400

Commit message: feat: start to routing DDR3
Parts:
- U101: footprint (none) -> Package_BGA:Xilinx_CLG400
Changed lines of the file:
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@@
 			)
 		)
-		(property "Footprint" ""
+		(property "Footprint" "Package_BGA:Xilinx_CLG400"
 			(at 215.9 316.23 0)
 			(hide yes)
@@
 			)
 		)
-		(property "Footprint" ""
+		(property "Footprint" "Package_BGA:Xilinx_CLG400"
 			(at 139.7 307.34 0)
 			(hide yes)
@@
 			)
 		)
-		(property "Footprint" ""
+		(property "Footprint" "Package_BGA:Xilinx_CLG400"
 			(at 82.55 340.36 0)
 			(hide yes)
@@
 			)
 		)
-		(property "Footprint" ""
+		(property "Footprint" "Package_BGA:Xilinx_CLG400"
 			(at 325.12 510.54 0)
 			(hide yes)
