File: ZYNQ_Pi_Zero.kicad_sch (KiCad schematic)
At the start: 1 part, among them U101 xc7z010clg400

Commit message: feat: continue sch design
Parts:
- removed U101: xc7z010clg400, Package_BGA:Xilinx_CLG400, symbol Xilinx7:xc7z010clg400
