File: ddr3.kicad_sch (KiCad schematic)
At the start: 22 parts, among them U101 xc7z010clg400, U201 MT41K256M16TW-107_P

Commit message: feat: continue routing ddr
Connections:
- net DDR_D0: now also U201.C3 (DQ9); no longer U201.C2 (DQ11)
- net DDR_D1: now also U201.A2 (DQ13); no longer U201.A3 (DQ15)
- net DDR_D2: now also U201.A3 (DQ15); no longer U201.A2 (DQ13)
- net DDR_D3: now also U201.C2 (DQ11); no longer U201.C3 (DQ9)
- net DDR_D4: now also U201.A7 (DQ12); no longer U201.D7 (DQ8)
- net DDR_D5: now also U201.C8 (DQ10); no longer U201.B8 (DQ14)
- net DDR_D6: now also U201.B8 (DQ14); no longer U201.C8 (DQ10)
- net DDR_D7: now also U201.D7 (DQ8); no longer U201.A7 (DQ12)
Changed lines of the file:
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@@
 	)
 	(label "DDR_D5"
-		(at 121.92 176.53 180)
+		(at 121.92 166.37 180)
 		(effects
 			(font
@@
 	)
 	(label "DDR_D1"
-		(at 121.92 179.07 180)
+		(at 121.92 173.99 180)
 		(effects
 			(font
@@
 	)
 	(label "DDR_D0"
-		(at 121.92 168.91 180)
+		(at 121.92 163.83 180)
 		(effects
 			(font
@@
 	)
 	(label "DDR_D7"
-		(at 121.92 171.45 180)
+		(at 121.92 161.29 180)
 		(effects
 			(font
@@
 	)
 	(label "DDR_D2"
-		(at 121.92 173.99 180)
+		(at 121.92 179.07 180)
 		(effects
 			(font
@@
 	)
 	(label "DDR_D3"
-		(at 121.92 163.83 180)
+		(at 121.92 168.91 180)
 		(effects
 			(font
@@
 	)
 	(label "DDR_D6"
-		(at 121.92 166.37 180)
+		(at 121.92 176.53 180)
 		(effects
 			(font
@@
 	)
 	(label "DDR_D4"
-		(at 121.92 161.29 180)
-		(effects
-			(font
+		(at 121.92 171.45 180)
+		(effects
+			(font
