File: ddr3.kicad_sch (KiCad schematic)
At the start: 46 parts, among them U101 xc7z010clg400, U201 MT41K256M16TW-107_P

Commit message: feat: continue routing
Parts:
- R206: footprint (none) -> Resistor_SMD:R_0402_1005Metric
Other:
- moved on the sheet: R202, R203, R206
Changed lines of the file:
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@@
 	)
 	(junction
-		(at 170.18 124.46)
+		(at 143.51 121.92)
 		(diameter 0)
 		(color 0 0 0 0)
@@
 	(wire
 		(pts
-			(xy 170.18 66.04) (xy 182.88 66.04)
+			(xy 146.05 64.77) (xy 158.75 64.77)
 		)
 		(stroke
@@
 	(wire
 		(pts
-			(xy 170.18 124.46) (xy 170.18 127)
+			(xy 143.51 121.92) (xy 143.51 124.46)
 		)
 		(stroke
@@
 	(wire
 		(pts
-			(xy 170.18 124.46) (xy 189.23 124.46)
+			(xy 143.51 121.92) (xy 162.56 121.92)
 		)
 		(stroke
@@
 	(wire
 		(pts
-			(xy 170.18 134.62) (xy 170.18 138.43)
+			(xy 143.51 132.08) (xy 143.51 135.89)
 		)
 		(stroke
@@
 	(wire
 		(pts
-			(xy 189.23 124.46) (xy 189.23 121.92)
+			(xy 162.56 121.92) (xy 162.56 119.38)
 		)
 		(stroke
@@
 	(wire
 		(pts
-			(xy 190.5 66.04) (xy 203.2 66.04)
+			(xy 166.37 64.77) (xy 179.07 64.77)
 		)
 		(stroke
@@
 	(wire
 		(pts
-			(xy 170.18 111.76) (xy 170.18 114.3)
+			(xy 143.51 109.22) (xy 143.51 111.76)
 		)
 		(stroke
@@
 	(wire
 		(pts
-			(xy 170.18 121.92) (xy 170.18 124.46)
+			(xy 143.51 119.38) (xy 143.51 121.92)
 		)
 		(stroke
@@
 	)
 	(label "DDR_CLK_P"
-		(at 203.2 66.04 180)
+		(at 179.07 64.77 180)
 		(effects
 			(font
@@
 	)
 	(label "DDR_CLK_N"
-		(at 170.18 66.04 0)
+		(at 146.05 64.77 0)
 		(effects
 			(font
@@
 	(symbol
 		(lib_id "power:+3V3")
-		(at 189.23 121.92 0)
+		(at 162.56 119.38 0)
 		(unit 1)
 		(body_style 1)
@@
 		(dnp no)
 		(property "Reference" "#PWR0222"
-			(at 189.23 125.73 0)
+			(at 162.56 123.19 0)
 			(hide yes)
 			(show_name no)
@@
 		)
 		(property "Value" "VTTREF"
-			(at 189.23 118.11 0)
+			(at 162.56 115.57 0)
 			(show_name no)
 			(do_not_autoplace no)
@@
 		)
 		(property "Footprint" ""
-			(at 189.23 121.92 0)
+			(at 162.56 119.38 0)
 			(hide yes)
 			(show_name no)
@@
 		)
 		(property "Datasheet" ""
-			(at 189.23 121.92 0)
+			(at 162.56 119.38 0)
 			(hide yes)
 			(show_name no)
@@
 		)
 		(property "Description" "Power symbol creates a global label with name \"+3V3\""
-			(at 189.23 121.92 0)
+			(at 162.56 119.38 0)
 			(hide yes)
 			(show_name no)
@@
 	(symbol
 		(lib_id "Device:R")
-		(at 186.69 66.04 90)
+		(at 162.56 64.77 90)
 		(unit 1)
 		(body_style 1)
@@
 		(dnp no)
 		(property "Reference" "R206"
-			(at 186.69 68.326 90)
+			(at 162.56 67.056 90)
 			(show_name no)
 			(do_not_autoplace no)
@@
 		)
 		(property "Value" "80R6"
-			(at 186.69 63.754 90)
+			(at 162.56 62.484 90)
 			(show_name no)
 			(do_not_autoplace no)
@@
 			)
 		)
-		(property "Footprint" ""
-			(at 186.69 67.818 90)
+		(property "Footprint" "Resistor_SMD:R_0402_1005Metric"
+			(at 162.56 66.548 90)
 			(hide yes)
 			(show_name no)
@@
 		)
 		(property "Datasheet" ""
-			(at 186.69 66.04 0)
+			(at 162.56 64.77 0)
 			(hide yes)
 			(show_name no)
@@
 		)
 		(property "Description" "Resistor"
-			(at 186.69 66.04 0)
+			(at 162.56 64.77 0)
 			(hide yes)
 			(show_name no)
@@
 	(symbol
 		(lib_id "Device:R")
-		(at 170.18 130.81 0)
+		(at 143.51 128.27 0)
 		(unit 1)
 		(body_style 1)
@@
 		(fields_autoplaced yes)
 		(property "Reference" "R203"
-			(at 172.72 129.5399 0)
+			(at 146.05 126.9999 0)
 			(show_name no)
 			(do_not_autoplace no)
@@
 		)
 		(property "Value" "10k"
-			(at 172.72 132.0799 0)
+			(at 146.05 129.5399 0)
 			(show_name no)
 			(do_not_autoplace no)
@@
 		)
 		(property "Footprint" "Resistor_SMD:R_0402_1005Metric"
-			(at 168.402 130.81 90)
+			(at 141.732 128.27 90)
 			(hide yes)
 			(show_name no)
@@
 		)
 		(property "Datasheet" ""
-			(at 170.18 130.81 0)
+			(at 143.51 128.27 0)
 			(hide yes)
 			(show_name no)
@@
 		)
 		(property "Description" "Resistor"
-			(at 170.18 130.81 0)
+			(at 143.51 128.27 0)
 			(hide yes)
 			(show_name no)
@@
 	(symbol
 		(lib_id "power:GND")
-		(at 170.18 138.43 0)
+		(at 143.51 135.89 0)
 		(unit 1)
 		(body_style 1)
@@
 		(dnp no)
 		(property "Reference" "#PWR0219"
-			(at 170.18 144.78 0)
+			(at 143.51 142.24 0)
 			(hide yes)
 			(show_name no)
@@
 		)
 		(property "Value" "GND"
-			(at 170.18 142.494 0)
+			(at 143.51 139.954 0)
 			(show_name no)
 			(do_not_autoplace no)
@@
 		)
 		(property "Footprint" ""
-			(at 170.18 138.43 0)
+			(at 143.51 135.89 0)
 			(hide yes)
 			(show_name no)
@@
 		)
 		(property "Datasheet" ""
-			(at 170.18 138.43 0)
+			(at 143.51 135.89 0)
 			(hide yes)
 			(show_name no)
@@
 		)
 		(property "Description" "Power symbol creates a global label with name \"GND\" , ground"
-			(at 170.18 138.43 0)
+			(at 143.51 135.89 0)
 			(hide yes)
 			(show_name no)
@@
 	(symbol
 		(lib_id "Device:R")
-		(at 170.18 118.11 0)
+		(at 143.51 115.57 0)
 		(unit 1)
 		(body_style 1)
@@
 		(fields_autoplaced yes)
 		(property "Reference" "R202"
-			(at 172.72 116.8399 0)
+			(at 146.05 114.2999 0)
 			(show_name no)
 			(do_not_autoplace no)
@@
 		)
 		(property "Value" "10k"
-			(at 172.72 119.3799 0)
+			(at 146.05 116.8399 0)
 			(show_name no)
 			(do_not_autoplace no)
@@
 		)
 		(property "Footprint" "Resistor_SMD:R_0402_1005Metric"
-			(at 168.402 118.11 90)
+			(at 141.732 115.57 90)
 			(hide yes)
 			(show_name no)
@@
 		)
 		(property "Datasheet" ""
-			(at 170.18 118.11 0)
+			(at 143.51 115.57 0)
 			(hide yes)
 			(show_name no)
@@
 		)
 		(property "Description" "Resistor"
-			(at 170.18 118.11 0)
+			(at 143.51 115.57 0)
 			(hide yes)
 			(show_name no)
@@
 	(symbol
 		(lib_id "power:+3V3")
-		(at 170.18 111.76 0)
+		(at 143.51 109.22 0)
 		(unit 1)
 		(body_style 1)
@@
 		(dnp no)
 		(property "Reference" "#PWR0218"
-			(at 170.18 115.57 0)
+			(at 143.51 113.03 0)
 			(hide yes)
 			(show_name no)
@@
 		)
 		(property "Value" "+1V5"
-			(at 170.18 107.95 0)
+			(at 143.51 105.41 0)
 			(show_name no)
 			(do_not_autoplace no)
@@
 		)
 		(property "Footprint" ""
-			(at 170.18 111.76 0)
+			(at 143.51 109.22 0)
 			(hide yes)
 			(show_name no)
@@
 		)
 		(property "Datasheet" ""
-			(at 170.18 111.76 0)
+			(at 143.51 109.22 0)
 			(hide yes)
 			(show_name no)
@@
 		)
 		(property "Description" "Power symbol creates a global label with name \"+3V3\""
-			(at 170.18 111.76 0)
+			(at 143.51 109.22 0)
 			(hide yes)
 			(show_name no)
