File: ZYNQ_Pi_Zero.kicad_pcb (KiCad board)
At the start: 4 copper layers, 35 parts, among them Q501 2N7002, Q502 2N7002, Q503 2N7002, U101 xc7z010clg400, U201 MT41K256M16TW-107_P, U301 W25Q256FVEI, U501 TPD4E05U06DQA, U502 TPD4E05U06DQA

Commit message: feat: continue routing ddr
Routing:
- net /DDR3/DDR_A7: track 11.9 -> 39.1 mm
- net /DDR3/DDR_A3: track 11.4 -> 36.5 mm
- net /DDR3/DDR_A9: track 11.2 -> 30.7 mm
- net /DDR3/DDR_A10: track 8.30 -> 23.3 mm
- net /DDR3/DDR_A11: track 13.3 -> 25.2 mm
- net /DDR3/DDR_BA1: track 9.18 -> 20.0 mm
- net /DDR3/DDR_ODT: track 3.23 -> 13.8 mm
- net /DDR3/DDR_~{WE}: track 1.47 -> 12.0 mm
- net /DDR3/DDR_A12: track 10.8 -> 21.2 mm
- net /DDR3/DDR_A5: track 12.8 -> 23.1 mm
- net /DDR3/DDR_A1: track 8.50 -> 18.7 mm
- net /DDR3/DDR_A8: track 6.46 -> 16.7 mm
- net /DDR3/DDR_A13: track 12.3 -> 22.4 mm
- net unconnected-(U101G-PS_DDR_DQ16_502-PadP1): track 3.57 -> 13.5 mm
- net /DDR3/DDR_~{CS}: track 5.69 -> 15.4 mm
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
Commit message: feat: continue routing ddr
Parts:
- moved C212 35.9 mm to (99.3, 95.3)
- moved C204 28.1 mm to (103.2, 105.6)
- moved C211 28.1 mm to (106.3, 105.7)
- moved C201 27.0 mm to (105.9, 88.9)
- moved C202 27.0 mm to (104.0, 88.9)
- moved C203 27.0 mm to (97.5, 88.9)
- moved C213 27.0 mm to (95.1, 88.9)
- moved C205 27.0 mm to (102.2, 88.9)
- moved C206 21.6 mm to (105.3, 104.5)
- moved R201 21.6 mm to (103.9, 104.5)
- moved C209 10.8 mm to (104.2, 101.3)
- moved C210 10.8 mm to (103.4, 102.5)
- moved C214 10.8 mm to (102.2, 101.3)
- moved R202 10.8 mm to (105.0, 97.8)
- moved R203 10.8 mm to (105.0, 96.8)
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Connections:
- U201 pad A2: /DDR3/DDR_D2 -> /DDR3/DDR_D1
- U201 pad A3: /DDR3/DDR_D1 -> /DDR3/DDR_D2
- U201 pad A7: /DDR3/DDR_D7 -> /DDR3/DDR_D4
- U201 pad B8: /DDR3/DDR_D5 -> /DDR3/DDR_D6
- U201 pad C2: /DDR3/DDR_D0 -> /DDR3/DDR_D3
- U201 pad C3: /DDR3/DDR_D3 -> /DDR3/DDR_D0
- U201 pad C8: /DDR3/DDR_D6 -> /DDR3/DDR_D5
- U201 pad D7: /DDR3/DDR_D4 -> /DDR3/DDR_D7
Routing:
- net /DDR3/DDR_A7: track 39.1 -> 0.00 mm, vias 2 -> 1
- net /DDR3/DDR_A3: track 36.5 -> 0.00 mm
- net /DDR3/DDR_A9: track 30.7 -> 0.00 mm
- net /DDR3/DDR_A11: track 25.2 -> 0.00 mm, vias 2 -> 1
- net /DDR3/DDR_A0: track 23.9 -> 0.00 mm
- net /DDR3/DDR_A5: track 23.1 -> 0.00 mm
- net /DDR3/DDR_A10: track 23.3 -> 0.57 mm, vias 2 -> 1
- net /DDR3/DDR_A13: track 22.4 -> 0.00 mm
- net /DDR3/DDR_A14: track 21.5 -> 0.00 mm, vias 2 -> 1
- net /DDR3/DDR_A12: track 21.2 -> 0.00 mm, vias 2 -> 1
- net /DDR3/DDR_BA1: track 20.0 -> 0.00 mm
- net /DDR3/DDR_CLK_N: track 21.0 -> 2.07 mm, vias 2 -> 1
- net /DDR3/DDR_A1: track 18.7 -> 0.00 mm, vias 1 -> 0
- net /DDR3/DDR_CLK_P: track 20.7 -> 2.07 mm, vias 2 -> 1
- net /DDR3/DDR_A2: track 18.4 -> 0.00 mm
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
Commit message: feat: continue routing ddr
Parts:
- moved U201 4.00 mm to (120.0, 100.0)
Connections:
- U201 pad A2: /DDR3/DDR_D1 -> /DDR3/DDR_D14
- U201 pad A3: /DDR3/DDR_D2 -> /DDR3/DDR_D9
- U201 pad A7: /DDR3/DDR_D4 -> /DDR3/DDR_D10
- U201 pad B8: /DDR3/DDR_D6 -> /DDR3/DDR_D11
- U201 pad C2: /DDR3/DDR_D3 -> /DDR3/DDR_D8
- U201 pad C3: /DDR3/DDR_D0 -> /DDR3/DDR_D13
- U201 pad C8: /DDR3/DDR_D5 -> /DDR3/DDR_D15
- U201 pad D7: /DDR3/DDR_D7 -> /DDR3/DDR_D12
- U201 pad E3: /DDR3/DDR_D8 -> /DDR3/DDR_D6
- U201 pad F2: /DDR3/DDR_D9 -> /DDR3/DDR_D3
- U201 pad F7: /DDR3/DDR_D11 -> /DDR3/DDR_D1
- U201 pad F8: /DDR3/DDR_D14 -> /DDR3/DDR_D0
- U201 pad G2: /DDR3/DDR_D13 -> /DDR3/DDR_D2
- U201 pad H3: /DDR3/DDR_D10 -> /DDR3/DDR_D5
- U201 pad H7: /DDR3/DDR_D15 -> /DDR3/DDR_D7
- U201 pad H8: /DDR3/DDR_D12 -> /DDR3/DDR_D4
Routing:
- net /DDR3/DDR_~{RESET}: track 0.00 -> 35.2 mm, vias 0 -> 2
- net /DDR3/DDR_DQS1_N: track 2.57 -> 30.5 mm, vias 1 -> 2
- net /DDR3/DDR_DQS1_P: track 2.57 -> 30.0 mm, vias 1 -> 2
- net /DDR3/DDR_D5: track 17.7 -> 36.9 mm
- net /DDR3/DDR_D8: track 15.8 -> 33.6 mm, vias 1 -> 0
- net /DDR3/DDR_D6: track 18.1 -> 35.5 mm
- net /DDR3/DDR_A3: track 0.00 -> 17.2 mm
- net /DDR3/DDR_A5: track 0.00 -> 15.3 mm
- net /DDR3/DDR_DQS0_N: track 20.7 -> 35.4 mm
- net /DDR3/DDR_D9: track 16.1 -> 30.3 mm
- net /DDR3/DDR_~{WE}: track 0.57 -> 14.7 mm
- net /DDR3/DDR_DQS0_P: track 20.8 -> 34.9 mm
- net /DDR3/DDR_BA2: track 0.57 -> 14.2 mm
- net /DDR3/DDR_D2: track 24.8 -> 38.3 mm, vias 0 -> 2
- net /DDR3/DDR_~{CS}: track 0.00 -> 13.5 mm
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