File: io.kicad_sch (KiCad schematic)
At the start: 1 part, among them U101 xc7z010clg400

Commit message: feat: modify sch design
Parts:
- removed U101: xc7z010clg400, Package_BGA:Xilinx_CLG400, symbol Xilinx7:xc7z010clg400
- added D801: LED, symbol Device:LED
- added R801: 1k, symbol Device:R
- added R802: 10k, symbol Device:R
- added R803: 100R, symbol Device:R
- added SW801: SW_Push, symbol Switch:SW_Push
- added U801: xc7z010clg400, Package_BGA:Xilinx_CLG400, symbol Xilinx7:xc7z010clg400
Connections:
- new net: D801.1 (K), R801.1
- new net: R802.2, R803.1, SW801.2
- new net +1V8: U801.C19 (VCCO_35[6]), U801.F18 (VCCO_35[6]), U801.H14 (VCCO_35[6]), U801.J17 (VCCO_35[6]), U801.K20 (VCCO_35[6]), U801.M16 (VCCO_35[6])
- new net +3V3: D801.2 (A), R802.1, U801.N19 (VCCO_34[6]), U801.R15 (VCCO_34[6]), U801.T18 (VCCO_34[6]), U801.V14 (VCCO_34[6]), U801.W17 (VCCO_34[6]), U801.Y20 (VCCO_34[6])
- new net GND: SW801.1
- new net PL_KEY1: R803.2
- new net PL_LED1: R801.2
Other:
- removed sheet BANK0
- removed sheet DDR3
- removed sheet HDMI
- removed sheet PL IO
- removed sheet POWER
- removed sheet PS MIO
- removed sheet SD CARD

Commit message: feat: continue routing ddr3
Parts:
- renumbered U801 to U101
Changed lines of the file:
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@@
 		(in_pos_files yes)
 		(dnp no)
-		(fields_autoplaced yes)
-		(property "Reference" "U801"
-			(at 205.74 55.8799 0)
+		(property "Reference" "U101"
+			(at 201.168 18.542 0)
 			(show_name no)
 			(do_not_autoplace no)
@@
 		)
 		(property "Value" "xc7z010clg400"
-			(at 205.74 58.4199 0)
+			(at 196.85 155.194 0)
 			(show_name no)
 			(do_not_autoplace no)
@@
 			(project "ZYNQ_Pi_Zero"
 				(path "/239d02af-7f9c-469f-b86b-abe2695ec54e/b946677b-d514-4782-808f-3d38ab75be74"
-					(reference "U801")
+					(reference "U101")
 					(unit 4)
 				)
@@
 		(dnp no)
 		(fields_autoplaced yes)
-		(property "Reference" "U801"
+		(property "Reference" "U101"
 			(at 135.89 160.02 90)
 			(show_name no)
@@
 			(project "ZYNQ_Pi_Zero"
 				(path "/239d02af-7f9c-469f-b86b-abe2695ec54e/b946677b-d514-4782-808f-3d38ab75be74"
-					(reference "U801")
+					(reference "U101")
 					(unit 9)
 				)
@@
 		(in_pos_files yes)
 		(dnp no)
-		(fields_autoplaced yes)
-		(property "Reference" "U801"
-			(at 123.19 55.8799 0)
+		(property "Reference" "U101"
+			(at 114.554 18.542 0)
 			(show_name no)
 			(do_not_autoplace no)
@@
 		)
 		(property "Value" "xc7z010clg400"
-			(at 123.19 58.4199 0)
+			(at 109.474 154.686 0)
 			(show_name no)
 			(do_not_autoplace no)
@@
 			(project "ZYNQ_Pi_Zero"
 				(path "/239d02af-7f9c-469f-b86b-abe2695ec54e/b946677b-d514-4782-808f-3d38ab75be74"
-					(reference "U801")
+					(reference "U101")
 					(unit 3)
 				)
@@
 		(in_pos_files yes)
 		(dnp no)
-		(property "Reference" "#PWR0802"
+		(property "Reference" "#PWR0801"
 			(at 22.86 92.71 0)
 			(hide yes)
@@
 			(project "ZYNQ_Pi_Zero"
 				(path "/239d02af-7f9c-469f-b86b-abe2695ec54e/b946677b-d514-4782-808f-3d38ab75be74"
-					(reference "#PWR0802")
+					(reference "#PWR0801")
 					(unit 1)
 				)
@@
 		(in_pos_files yes)
 		(dnp no)
-		(property "Reference" "#PWR0806"
+		(property "Reference" "#PWR0804"
 			(at 43.18 149.86 0)
 			(hide yes)
@@
 			(project "ZYNQ_Pi_Zero"
 				(path "/239d02af-7f9c-469f-b86b-abe2695ec54e/b946677b-d514-4782-808f-3d38ab75be74"
-					(reference "#PWR0806")
+					(reference "#PWR0804")
 					(unit 1)
 				)
@@
 		(in_pos_files yes)
 		(dnp no)
-		(property "Reference" "#PWR0808"
+		(property "Reference" "#PWR0805"
 			(at 43.18 158.75 0)
 			(hide yes)
@@
 			(project "ZYNQ_Pi_Zero"
 				(path "/239d02af-7f9c-469f-b86b-abe2695ec54e/b946677b-d514-4782-808f-3d38ab75be74"
-					(reference "#PWR0808")
+					(reference "#PWR0805")
 					(unit 1)
 				)
@@
 		(in_pos_files yes)
 		(dnp no)
-		(property "Reference" "#PWR0809"
+		(property "Reference" "#PWR0807"
 			(at 57.15 158.75 0)
 			(hide yes)
@@
 			(project "ZYNQ_Pi_Zero"
 				(path "/239d02af-7f9c-469f-b86b-abe2695ec54e/b946677b-d514-4782-808f-3d38ab75be74"
-					(reference "#PWR0809")
+					(reference "#PWR0807")
 					(unit 1)
 				)
@@
 		(in_pos_files yes)
 		(dnp no)
-		(property "Reference" "#PWR0801"
+		(property "Reference" "#PWR0802"
 			(at 36.83 34.29 0)
 			(hide yes)
@@
 			(project "ZYNQ_Pi_Zero"
 				(path "/239d02af-7f9c-469f-b86b-abe2695ec54e/b946677b-d514-4782-808f-3d38ab75be74"
-					(reference "#PWR0801")
+					(reference "#PWR0802")
 					(unit 1)
 				)
@@
 		(in_pos_files yes)
 		(dnp no)
-		(property "Reference" "#PWR0804"
+		(property "Reference" "#PWR0808"
 			(at 85.09 148.59 0)
 			(hide yes)
@@
 			(project "ZYNQ_Pi_Zero"
 				(path "/239d02af-7f9c-469f-b86b-abe2695ec54e/b946677b-d514-4782-808f-3d38ab75be74"
-					(reference "#PWR0804")
+					(reference "#PWR0808")
 					(unit 1)
 				)
@@
 		(in_pos_files yes)
 		(dnp no)
-		(property "Reference" "#PWR0805"
+		(property "Reference" "#PWR0809"
 			(at 168.91 148.59 0)
 			(hide yes)
@@
 			(project "ZYNQ_Pi_Zero"
 				(path "/239d02af-7f9c-469f-b86b-abe2695ec54e/b946677b-d514-4782-808f-3d38ab75be74"
-					(reference "#PWR0805")
+					(reference "#PWR0809")
 					(unit 1)
 				)
@@
 		(in_pos_files yes)
 		(dnp no)
-		(property "Reference" "#PWR0807"
+		(property "Reference" "#PWR0806"
 			(at 57.15 149.86 0)
 			(hide yes)
@@
 			(project "ZYNQ_Pi_Zero"
 				(path "/239d02af-7f9c-469f-b86b-abe2695ec54e/b946677b-d514-4782-808f-3d38ab75be74"
-					(reference "#PWR0807")
+					(reference "#PWR0806")
 					(unit 1)
 				)

Commit message: feat: continue routing
Parts:
- D801: footprint (none) -> LED_SMD:LED_0603_1608Metric
- R801: footprint (none) -> Resistor_SMD:R_0402_1005Metric
Changed lines of the file:
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@@
 			)
 		)
-		(property "Footprint" ""
+		(property "Footprint" "Resistor_SMD:R_0402_1005Metric"
 			(at 35.052 48.26 90)
 			(hide yes)
@@
 			)
 		)
-		(property "Footprint" ""
+		(property "Footprint" "LED_SMD:LED_0603_1608Metric"
 			(at 36.83 36.83 0)
 			(hide yes)
