File: power.kicad_sch (KiCad schematic)
At the start: 32 parts, among them U101 xc7z010clg400, U401 TPS621351, U402 TLV62130RGTT, U403 TLV62130RGTT, U404 SPX3819M5-L-3-3

Commit message: feat: continue sch design
Parts:
- added J401: USB_C_Receptacle_USB2.0_16P, symbol Connector:USB_C_Receptacle_USB2.0_16P
- added R410, R411: 5k1, symbol Device:R
- added U405: xc7z010clg400, Package_BGA:Xilinx_CLG400, symbol Xilinx7:xc7z010clg400
Connections:
- net +3V3: now also U405.T8 (VCCO_13[4]), U405.U11 (VCCO_13[4]), U405.W7 (VCCO_13[4]), U405.Y10 (VCCO_13[4])
- net +5V: now also J401.A4 (VBUS), J401.A9 (VBUS), J401.B4 (VBUS), J401.B9 (VBUS)
- net GND: now also J401.A1 (GND), J401.A12 (GND), J401.B1 (GND), J401.B12 (GND), J401.SH (SHIELD), R410.2, R411.2
- new net: J401.A5 (CC1), R410.1
- new net: J401.B5 (CC2), R411.1
- new net USB_D+: J401.A6 (D+), J401.B6 (D+)
- new net USB_D-: J401.A7 (D-), J401.B7 (D-)
- no-connect marks 1 -> 3
Other:
- moved on the sheet: C401, C402, C403, C404, C405, C406, C407, C408, C409, C410, C411, C412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

Commit message: feat: continue routing ddr3
Parts:
- added C409, C410, C416, C417, C420, C421, C425, C426, C432, C433: 4u7, Capacitor_SMD:C_0603_1608Metric, symbol Device:C
- added C411, C412, C418, C419, C422, C423, C424, C427, C428, C429, C434, C435: 470n, Capacitor_SMD:C_0402_1005Metric, symbol Device:C
- C401, C402: footprint (none) -> Capacitor_SMD:C_0805_2012Metric
- C403, C404: footprint (none) -> Capacitor_SMD:C_0402_1005Metric
- C405: renamed from C407; footprint (none) -> Capacitor_SMD:C_0805_2012Metric
- C406: renamed from C411; footprint (none) -> Capacitor_SMD:C_0805_2012Metric
- C407: renamed from C408; footprint (none) -> Capacitor_SMD:C_0805_2012Metric
- C408: renamed from C409; footprint (none) -> Capacitor_SMD:C_0805_2012Metric
- C413: renamed from C412; footprint (none) -> Capacitor_SMD:C_0805_2012Metric
- C414: renamed from C410; footprint (none) -> Capacitor_SMD:C_0402_1005Metric
- C430: renamed from C405; footprint (none) -> Capacitor_SMD:C_0805_2012Metric
- C431: renamed from C406; footprint (none) -> Capacitor_SMD:C_0402_1005Metric
- C436: renamed from C414; footprint (none) -> Capacitor_SMD:C_0805_2012Metric
- U404: PACKAGE SOT-23-5 -> (none)
- renumbered C413 to C415, R411 to R402, R410 to R403, R402 to R404, R403 to R405, R404 to R406, R405 to R407, R406 to R408, R407 to R409, R408 to R410, R409 to R411, U405 to U101, U403 to U405
Connections:
- net +1V0: now also C409.1, C411.1, C420.1, C422.1, C424.1, C425.1, C427.1, C429.1
- net +1V5: now also C433.1, C435.1
- net +1V8: now also C416.1, C418.1, C426.1, C428.1, C432.1, C434.1
- net +3V3: now also C421.1, C423.1
- net GND: now also C409.2, C410.2, C411.2, C412.2, C416.2, C417.2, C418.2, C419.2, C420.2, C421.2, C422.2, C423.2, C424.2, C425.2, C426.2, C427.2, C428.2, C429.2, C432.2, C433.2, C434.2, C435.2
- new net VCCIO_34: C410.1, C412.1
- new net VCCIO_35: C417.1, C419.1
Other:
- note added: "VCCAUX"
- note added: "VCCBRAM"
- note added: "VCCINT"
- note added: "VCCO_DDR_502"
- note added: "VCCO_MIO0_500"
- note added: "VCCO_MIO0_501"
- note added: "VCCPAUX"
- note added: "VCCPINT"
- note added: "VCC_34"
- note added: "VCC_35"
- moved on the sheet: C401, C402, C403, C404, C405, C406, C407, C413, C415, C430, C431, FB401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

Commit message: feat: continue routing
Parts:
- R401, R402, R403, R405, R406, R407, R408, R410, R411: footprint (none) -> Resistor_SMD:R_0402_1005Metric
Changed lines of the file:
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@@
 			)
 		)
-		(property "Footprint" ""
+		(property "Footprint" "Resistor_SMD:R_0402_1005Metric"
 			(at 101.092 43.18 90)
 			(hide yes)
@@
 			)
 		)
-		(property "Footprint" ""
+		(property "Footprint" "Resistor_SMD:R_0402_1005Metric"
 			(at 247.142 38.1 90)
 			(hide yes)
@@
 			)
 		)
-		(property "Footprint" ""
+		(property "Footprint" "Resistor_SMD:R_0402_1005Metric"
 			(at 247.142 48.26 90)
 			(hide yes)
@@
 			)
 		)
-		(property "Package" "SOT-23-5"
-			(at 144.78 173.99 0)
-			(hide yes)
-			(show_name no)
-			(do_not_autoplace no)
-			(effects
-				(font
-					(size 1.27 1.27)
-				)
-				(justify bottom)
-			)
-		)
 		(property "MPN" "SPX3819M5-L-3-3"
 			(at 144.78 173.99 0)
@@
 			)
 		)
-		(property "Footprint" ""
+		(property "Footprint" "Resistor_SMD:R_0402_1005Metric"
 			(at 82.55 44.958 90)
 			(hide yes)
@@
 			)
 		)
-		(property "Footprint" ""
+		(property "Footprint" "Resistor_SMD:R_0402_1005Metric"
 			(at 95.758 161.29 90)
 			(hide yes)
@@
 			)
 		)
-		(property "Footprint" ""
+		(property "Footprint" "Resistor_SMD:R_0402_1005Metric"
 			(at 116.332 105.41 90)
 			(hide yes)
@@
 			)
 		)
-		(property "Footprint" ""
+		(property "Footprint" "Resistor_SMD:R_0402_1005Metric"
 			(at 101.092 53.34 90)
 			(hide yes)
@@
 			)
 		)
-		(property "Footprint" ""
+		(property "Footprint" "Resistor_SMD:R_0402_1005Metric"
 			(at 116.332 95.25 90)
 			(hide yes)
@@
 			)
 		)
-		(property "Footprint" ""
+		(property "Footprint" "Resistor_SMD:R_0402_1005Metric"
 			(at 96.012 161.29 90)
 			(hide yes)
