File: mio.kicad_sch (KiCad schematic)
At the start: 1 part, among them U101 xc7z010clg400

Commit message: feat: finish ddr3 sch design
Parts:
- removed U101: xc7z010clg400, symbol Xilinx7:xc7z010clg400
- added C701: 470n, symbol Device:C
- added R701, R702: 33R, symbol Device:R
- added R703, R704: 1k, symbol Device:R
- added U701: xc7z010clg400, symbol Xilinx7:xc7z010clg400
Connections:
- new net: R702.2, U701.A5 (PS_MIO6_500)
- new net: C701.1, R703.2, R704.1, U701.E11 (PS_MIO_VREF_501)
- new net: R701.2, U701.D14 (PS_MIO40_501)
- new net +1V8: R703.1, U701.A13 (VCCO_MIO1_501[4]), U701.B16 (VCCO_MIO1_501[4]), U701.D12 (VCCO_MIO1_501[4]), U701.E15 (VCCO_MIO1_501[4])
- new net +3V3: U701.B6 (VCCO_MIO0_500[2]), U701.D7 (VCCO_MIO0_500[2])
- new net GND: C701.2, R704.2
- new net PS_CLK: U701.E7 (PS_CLK_500)
- new net PS_MIO0: U701.E6 (PS_MIO0_500)
- new net PS_MIO10: U701.E9 (PS_MIO10_500)
- new net PS_MIO11: U701.C6 (PS_MIO11_500)
- new net PS_MIO12: U701.D9 (PS_MIO12_500)
- new net PS_MIO13: U701.E8 (PS_MIO13_500)
- new net PS_MIO14: U701.C5 (PS_MIO14_500)
- new net PS_MIO15: U701.C8 (PS_MIO15_500)
- new net PS_MIO7: U701.D8 (PS_MIO7_500)
- new net PS_MIO8: U701.D5 (PS_MIO8_500)
- new net PS_MIO9: U701.B5 (PS_MIO9_500)
- new net PS_POR_B: U701.C7 (PS_POR_B_500)
- new net PS_SRST_B: U701.B10 (PS_SRST_B_501)
- new net QSPI_CLK: R702.1
- new net QSPI_CS: U701.A7 (PS_MIO1_500)
- new net QSPI_D0: U701.B8 (PS_MIO2_500)
- new net QSPI_D1: U701.D6 (PS_MIO3_500)
- new net QSPI_D2_PS_MIO4: U701.B7 (PS_MIO4_500)
- new net QSPI_D3_PS_MIO5: U701.A6 (PS_MIO5_500)
- new net SD_CLK: R701.1
- new net SD_CMD: U701.C17 (PS_MIO41_501)
- new net SD_DATA0: U701.E12 (PS_MIO42_501)
- new net SD_DATA1: U701.A9 (PS_MIO43_501)
- new net SD_DATA2: U701.F13 (PS_MIO44_501)
- new net SD_DATA3: U701.B15 (PS_MIO45_501)
Other:
- removed sheet BANK0
- removed sheet DDR3
- removed sheet HDMI
- removed sheet POWER
- removed sheet PS MIO
- removed sheet SD CARD

Commit message: feat: restart routing ddr
Parts:
- renumbered R702 to R701, R703 to R702, R704 to R703, R701 to R704
Changed lines of the file:
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@@
 		(in_pos_files yes)
 		(dnp no)
-		(property "Reference" "R702"
+		(property "Reference" "R701"
 			(at 59.69 96.52 90)
 			(show_name no)
@@
 			(project "ZYNQ_Pi_Zero"
 				(path "/239d02af-7f9c-469f-b86b-abe2695ec54e/e2d55b2b-db37-4002-990c-3c8d9a3ba028"
-					(reference "R702")
+					(reference "R701")
 					(unit 1)
 				)
@@
 		(in_pos_files yes)
 		(dnp no)
-		(property "Reference" "#PWR0704"
+		(property "Reference" "#PWR0702"
 			(at 198.12 130.81 0)
 			(hide yes)
@@
 			(project "ZYNQ_Pi_Zero"
 				(path "/239d02af-7f9c-469f-b86b-abe2695ec54e/e2d55b2b-db37-4002-990c-3c8d9a3ba028"
-					(reference "#PWR0704")
+					(reference "#PWR0702")
 					(unit 1)
 				)
@@
 		(dnp no)
 		(fields_autoplaced yes)
-		(property "Reference" "R703"
+		(property "Reference" "R702"
 			(at 200.66 132.0799 0)
 			(show_name no)
@@
 			(project "ZYNQ_Pi_Zero"
 				(path "/239d02af-7f9c-469f-b86b-abe2695ec54e/e2d55b2b-db37-4002-990c-3c8d9a3ba028"
-					(reference "R703")
+					(reference "R702")
 					(unit 1)
 				)
@@
 		(dnp no)
 		(fields_autoplaced yes)
-		(property "Reference" "R704"
+		(property "Reference" "R703"
 			(at 200.66 142.2399 0)
 			(show_name no)
@@
 			(project "ZYNQ_Pi_Zero"
 				(path "/239d02af-7f9c-469f-b86b-abe2695ec54e/e2d55b2b-db37-4002-990c-3c8d9a3ba028"
-					(reference "R704")
+					(reference "R703")
 					(unit 1)
 				)
@@
 		(in_pos_files yes)
 		(dnp no)
-		(property "Reference" "R701"
+		(property "Reference" "R704"
 			(at 216.662 101.6 90)
 			(show_name no)
@@
 			(project "ZYNQ_Pi_Zero"
 				(path "/239d02af-7f9c-469f-b86b-abe2695ec54e/e2d55b2b-db37-4002-990c-3c8d9a3ba028"
-					(reference "R701")
+					(reference "R704")
 					(unit 1)
 				)
@@
 		(in_pos_files yes)
 		(dnp no)
-		(property "Reference" "#PWR0702"
+		(property "Reference" "#PWR0704"
 			(at 210.82 130.81 0)
 			(hide yes)
@@
 			(project "ZYNQ_Pi_Zero"
 				(path "/239d02af-7f9c-469f-b86b-abe2695ec54e/e2d55b2b-db37-4002-990c-3c8d9a3ba028"
-					(reference "#PWR0702")
+					(reference "#PWR0704")
 					(unit 1)
 				)

Commit message: feat: modify sch design
Parts:
- added C702: 100n, symbol Device:C
- added D701: LED, symbol Device:LED
- added R705: 1k, symbol Device:R
- added R706, R708, R711: 10k, symbol Device:R
- added R707, R709: 100R, symbol Device:R
- added R710: 33R, symbol Device:R
- added SW701, SW702: SW_Push, symbol Switch:SW_Push
- added U702: 33.3333MHz, Oscillator:Oscillator_SMD_SeikoEpson_SG8002CE-4Pin_3.2x2.5mm, symbol Osc33.3333MHz:EPSON_Q33310F700622
Connections:
- net +1V8: now also R711.1
- net +3V3: now also C702.1, D701.2 (A), R706.1, R708.1, U702.1 (OE), U702.4 (VDD)
- net GND: now also C702.2, SW701.1, SW702.1, U702.2 (GND)
- net PS_CLK: now also R710.2
- net PS_POR_B: now also R709.2
- net PS_SRST_B: now also R711.2
- new net: D701.1 (K), R705.1
- new net: R710.1, U702.3 (OUT)
- new net: R708.2, R709.1, SW702.2
- new net: R706.2, R707.1, SW701.2
- new net PS_KEY1: R707.2
- new net PS_LED1: R705.2
Other:
- moved on the sheet: R701, U701E

Commit message: feat: continue routing ddr3
Parts:
- C701: renamed from C702; footprint (none) -> Capacitor_SMD:C_0402_1005Metric
- C702: renamed from C701; footprint (none) -> Capacitor_SMD:C_0402_1005Metric
- renumbered R705 to R701, R706 to R702, R707 to R703, R701 to R704, R708 to R705, R709 to R706, R710 to R707, R702 to R708, R703 to R709, R711 to R710, R704 to R711, U701 to U101
Changed lines of the file:
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@@
 		(in_pos_files yes)
 		(dnp no)
-		(property "Reference" "#PWR0708"
+		(property "Reference" "#PWR0707"
 			(at 115.57 57.15 0)
 			(hide yes)
@@
 			(project "ZYNQ_Pi_Zero"
 				(path "/239d02af-7f9c-469f-b86b-abe2695ec54e/e2d55b2b-db37-4002-990c-3c8d9a3ba028"
-					(reference "#PWR0708")
+					(reference "#PWR0707")
 					(unit 1)
 				)
@@
 		(in_pos_files yes)
 		(dnp no)
-		(property "Reference" "R701"
+		(property "Reference" "R704"
 			(at 101.6 96.52 90)
 			(show_name no)
@@
 			(project "ZYNQ_Pi_Zero"
 				(path "/239d02af-7f9c-469f-b86b-abe2695ec54e/e2d55b2b-db37-4002-990c-3c8d9a3ba028"
-					(reference "R701")
+					(reference "R704")
 					(unit 1)
 				)
@@
 		(in_pos_files yes)
 		(dnp no)
-		(property "Reference" "#PWR0705"
+		(property "Reference" "#PWR0701"
 			(at 39.37 35.56 0)
 			(hide yes)
@@
 			(project "ZYNQ_Pi_Zero"
 				(path "/239d02af-7f9c-469f-b86b-abe2695ec54e/e2d55b2b-db37-4002-990c-3c8d9a3ba028"
-					(reference "#PWR0705")
+					(reference "#PWR0701")
 					(unit 1)
 				)
@@
 		(in_pos_files yes)
 		(dnp no)
-		(property "Reference" "#PWR0702"
+		(property "Reference" "#PWR0709"
 			(at 198.12 130.81 0)
 			(hide yes)
@@
 			(project "ZYNQ_Pi_Zero"
 				(path "/239d02af-7f9c-469f-b86b-abe2695ec54e/e2d55b2b-db37-4002-990c-3c8d9a3ba028"
-					(reference "#PWR0702")
+					(reference "#PWR0709")
 					(unit 1)
 				)
@@
 		(in_pos_files yes)
 		(dnp no)
-		(property "Reference" "#PWR0703"
+		(property "Reference" "#PWR0710"
 			(at 198.12 157.48 0)
 			(hide yes)
@@
 			(project "ZYNQ_Pi_Zero"
 				(path "/239d02af-7f9c-469f-b86b-abe2695ec54e/e2d55b2b-db37-4002-990c-3c8d9a3ba028"
-					(reference "#PWR0703")
+					(reference "#PWR0710")
 					(unit 1)
 				)
@@
 		(dnp no)
 		(fields_autoplaced yes)
-		(property "Reference" "R702"
+		(property "Reference" "R708"
 			(at 200.66 132.0799 0)
 			(show_name no)
@@
 			(project "ZYNQ_Pi_Zero"
 				(path "/239d02af-7f9c-469f-b86b-abe2695ec54e/e2d55b2b-db37-4002-990c-3c8d9a3ba028"
-					(reference "R702")
+					(reference "R708")
 					(unit 1)
 				)
@@
 		(in_pos_files yes)
 		(dnp no)
-		(property "Reference" "#PWR0701"
+		(property "Reference" "#PWR0703"
 			(at 77.47 127 0)
 			(hide yes)
@@
 			(project "ZYNQ_Pi_Zero"
 				(path "/239d02af-7f9c-469f-b86b-abe2695ec54e/e2d55b2b-db37-4002-990c-3c8d9a3ba028"
-					(reference "#PWR0701")
+					(reference "#PWR0703")
 					(unit 1)
 				)
@@
 		(in_pos_files yes)
 		(dnp no)
-		(property "Reference" "C701"
+		(property "Reference" "C702"
 			(at 187.96 142.2399 0)
 			(show_name no)
@@
 			)
 		)
-		(property "Footprint" ""
+		(property "Footprint" "Capacitor_SMD:C_0402_1005Metric"
 			(at 190.8048 147.32 0)
 			(hide yes)
@@
 			(project "ZYNQ_Pi_Zero"
 				(path "/239d02af-7f9c-469f-b86b-abe2695ec54e/e2d55b2b-db37-4002-990c-3c8d9a3ba028"
-					(reference "C701")
+					(reference "C702")
 					(unit 1)
 				)
@@
 		(in_pos_files yes)
 		(dnp no)
-		(property "Reference" "U701"
+		(property "Reference" "U101"
 			(at 246.634 37.592 0)
 			(show_name no)
@@
 			(project "ZYNQ_Pi_Zero"
 				(path "/239d02af-7f9c-469f-b86b-abe2695ec54e/e2d55b2b-db37-4002-990c-3c8d9a3ba028"
-					(reference "U701")
+					(reference "U101")
 					(unit 6)
 				)
@@
 		(dnp no)
 		(fields_autoplaced yes)
-		(property "Reference" "R703"
+		(property "Reference" "R709"
 			(at 200.66 142.2399 0)
 			(show_name no)
@@
 			(project "ZYNQ_Pi_Zero"
 				(path "/239d02af-7f9c-469f-b86b-abe2695ec54e/e2d55b2b-db37-4002-990c-3c8d9a3ba028"
-					(reference "R703")
+					(reference "R709")
 					(unit 1)
 				)
@@
 		(in_pos_files yes)
 		(dnp no)
-		(property "Reference" "R710"
+		(property "Reference" "R707"
 			(at 138.43 167.64 90)
 			(show_name no)
@@
 			(project "ZYNQ_Pi_Zero"
 				(path "/239d02af-7f9c-469f-b86b-abe2695ec54e/e2d55b2b-db37-4002-990c-3c8d9a3ba028"
-					(reference "R710")
+					(reference "R707")
 					(unit 1)
 				)
@@
 		(in_pos_files yes)
 		(dnp no)
-		(property "Reference" "R709"
+		(property "Reference" "R706"
 			(at 142.24 54.61 90)
 			(show_name no)
@@
 			(project "ZYNQ_Pi_Zero"
 				(path "/239d02af-7f9c-469f-b86b-abe2695ec54e/e2d55b2b-db37-4002-990c-3c8d9a3ba028"
-					(reference "R709")
+					(reference "R706")
 					(unit 1)
 				)
@@
 		(in_pos_files yes)
 		(dnp no)
-		(property "Reference" "R707"
+		(property "Reference" "R703"
 			(at 87.63 54.61 90)
 			(show_name no)
@@
 			(project "ZYNQ_Pi_Zero"
 				(path "/239d02af-7f9c-469f-b86b-abe2695ec54e/e2d55b2b-db37-4002-990c-3c8d9a3ba028"
-					(reference "R707")
+					(reference "R703")
 					(unit 1)
 				)
@@
 		(in_pos_files yes)
 		(dnp no)
-		(property "Reference" "R704"
+		(property "Reference" "R711"
 			(at 216.662 101.6 90)
 			(show_name no)
@@
 			(project "ZYNQ_Pi_Zero"
 				(path "/239d02af-7f9c-469f-b86b-abe2695ec54e/e2d55b2b-db37-4002-990c-3c8d9a3ba028"
-					(reference "R704")
+					(reference "R711")
 					(unit 1)
 				)
@@
 		(in_pos_files yes)
 		(dnp no)
-		(property "Reference" "#PWR0711"
+		(property "Reference" "#PWR0706"
 			(at 114.3 153.67 0)
 			(hide yes)
@@
 			(project "ZYNQ_Pi_Zero"
 				(path "/239d02af-7f9c-469f-b86b-abe2695ec54e/e2d55b2b-db37-4002-990c-3c8d9a3ba028"
-					(reference "#PWR0711")
+					(reference "#PWR0706")
 					(unit 1)
 				)
@@
 		(in_pos_files yes)
 		(dnp no)
-		(property "Reference" "#PWR0707"
+		(property "Reference" "#PWR0702"
 			(at 60.96 57.15 0)
 			(hide yes)
@@
 			(project "ZYNQ_Pi_Zero"
 				(path "/239d02af-7f9c-469f-b86b-abe2695ec54e/e2d55b2b-db37-4002-990c-3c8d9a3ba028"
-					(reference "#PWR0707")
+					(reference "#PWR0702")
 					(unit 1)
 				)
@@
 		(dnp no)
 		(fields_autoplaced yes)
-		(property "Reference" "R711"
+		(property "Reference" "R710"
 			(at 218.44 76.1999 0)
 			(show_name no)
@@
 			(project "ZYNQ_Pi_Zero"
 				(path "/239d02af-7f9c-469f-b86b-abe2695ec54e/e2d55b2b-db37-4002-990c-3c8d9a3ba028"
-					(reference "R711")
+					(reference "R710")
 					(unit 1)
 				)
@@
 		(in_pos_files yes)
 		(dnp no)
-		(property "Reference" "C702"
+		(property "Reference" "C701"
 			(at 105.41 161.2899 0)
 			(show_name no)
@@
 			)
 		)
-		(property "Footprint" ""
+		(property "Footprint" "Capacitor_SMD:C_0402_1005Metric"
 			(at 108.2548 166.37 0)
 			(hide yes)
@@
 			(project "ZYNQ_Pi_Zero"
 				(path "/239d02af-7f9c-469f-b86b-abe2695ec54e/e2d55b2b-db37-4002-990c-3c8d9a3ba028"
-					(reference "C702")
+					(reference "C701")
 					(unit 1)
 				)
@@
 		(in_pos_files yes)
 		(dnp no)
-		(property "Reference" "U701"
+		(property "Reference" "U101"
 			(at 127 75.946 0)
 			(show_name no)
@@
 			(project "ZYNQ_Pi_Zero"
 				(path "/239d02af-7f9c-469f-b86b-abe2695ec54e/e2d55b2b-db37-4002-990c-3c8d9a3ba028"
-					(reference "U701")
+					(reference "U101")
 					(unit 5)
 				)
@@
 		(in_pos_files yes)
 		(dnp no)
-		(property "Reference" "#PWR0704"
+		(property "Reference" "#PWR0711"
 			(at 210.82 130.81 0)
 			(hide yes)
@@
 			(project "ZYNQ_Pi_Zero"
 				(path "/239d02af-7f9c-469f-b86b-abe2695ec54e/e2d55b2b-db37-4002-990c-3c8d9a3ba028"
-					(reference "#PWR0704")
+					(reference "#PWR0711")
 					(unit 1)
 				)
@@
 		(in_pos_files yes)
 		(dnp no)
-		(property "Reference" "#PWR0706"
+		(property "Reference" "#PWR0704"
 			(at 80.01 35.56 0)
 			(hide yes)
@@
 			(project "ZYNQ_Pi_Zero"
 				(path "/239d02af-7f9c-469f-b86b-abe2695ec54e/e2d55b2b-db37-4002-990c-3c8d9a3ba028"
-					(reference "#PWR0706")
+					(reference "#PWR0704")
 					(unit 1)
 				)
@@
 		(in_pos_files yes)
 		(dnp no)
-		(property "Reference" "#PWR0709"
+		(property "Reference" "#PWR0708"
 			(at 134.62 35.56 0)
 			(hide yes)
@@
 			(project "ZYNQ_Pi_Zero"
 				(path "/239d02af-7f9c-469f-b86b-abe2695ec54e/e2d55b2b-db37-4002-990c-3c8d9a3ba028"
-					(reference "#PWR0709")
+					(reference "#PWR0708")
 					(unit 1)
 				)
@@
 		(dnp no)
 		(fields_autoplaced yes)
-		(property "Reference" "R705"
+		(property "Reference" "R701"
 			(at 41.91 48.2599 0)
 			(show_name no)
@@
 			(project "ZYNQ_Pi_Zero"
 				(path "/239d02af-7f9c-469f-b86b-abe2695ec54e/e2d55b2b-db37-4002-990c-3c8d9a3ba028"
-					(reference "R705")
+					(reference "R701")
 					(unit 1)
 				)
@@
 		(dnp no)
 		(fields_autoplaced yes)
-		(property "Reference" "R708"
+		(property "Reference" "R705"
 			(at 137.16 36.8299 0)
 			(show_name no)
@@
 			(project "ZYNQ_Pi_Zero"
 				(path "/239d02af-7f9c-469f-b86b-abe2695ec54e/e2d55b2b-db37-4002-990c-3c8d9a3ba028"
-					(reference "R708")
+					(reference "R705")
 					(unit 1)
 				)
@@
 		(dnp no)
 		(fields_autoplaced yes)
-		(property "Reference" "R706"
+		(property "Reference" "R702"
 			(at 82.55 36.8299 0)
 			(show_name no)
@@
 			(project "ZYNQ_Pi_Zero"
 				(path "/239d02af-7f9c-469f-b86b-abe2695ec54e/e2d55b2b-db37-4002-990c-3c8d9a3ba028"
-					(reference "R706")
+					(reference "R702")
 					(unit 1)
 				)
@@
 		(in_pos_files yes)
 		(dnp no)
-		(property "Reference" "#PWR0710"
+		(property "Reference" "#PWR0705"
 			(at 109.22 179.07 0)
 			(hide yes)
@@
 			(project "ZYNQ_Pi_Zero"
 				(path "/239d02af-7f9c-469f-b86b-abe2695ec54e/e2d55b2b-db37-4002-990c-3c8d9a3ba028"
-					(reference "#PWR0710")
+					(reference "#PWR0705")
 					(unit 1)
 				)

Commit message: feat: continue routing
Parts:
- D701: footprint (none) -> LED_SMD:LED_0603_1608Metric
- R701, R708, R709: footprint (none) -> Resistor_SMD:R_0402_1005Metric
Changed lines of the file:
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@@
 			)
 		)
-		(property "Footprint" ""
+		(property "Footprint" "LED_SMD:LED_0603_1608Metric"
 			(at 39.37 38.1 0)
 			(hide yes)
@@
 			)
 		)
-		(property "Footprint" ""
+		(property "Footprint" "Resistor_SMD:R_0402_1005Metric"
 			(at 199.898 133.35 90)
 			(hide yes)
@@
 			)
 		)
-		(property "Footprint" ""
+		(property "Footprint" "Resistor_SMD:R_0402_1005Metric"
 			(at 199.898 143.51 90)
 			(hide yes)
@@
 			)
 		)
-		(property "Footprint" ""
+		(property "Footprint" "Resistor_SMD:R_0402_1005Metric"
 			(at 37.592 49.53 90)
 			(hide yes)

Commit message: feat: add sd card footprint
Parts:
- R711: footprint (none) -> Resistor_SMD:R_0402_1005Metric
Changed lines of the file:
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@@
 			)
 		)
-		(property "Footprint" ""
+		(property "Footprint" "Resistor_SMD:R_0402_1005Metric"
 			(at 222.25 104.648 90)
 			(hide yes)
@@
 		)
 	)
+	(group ""
+		(members "0bf38251-e84c-4b2e-800d-c983d5ccd16d" "1e83c2ad-b3fd-426c-ad25-351ea102476b"
+			"262f66d1-add9-4908-a9d0-4241472963fd" "9d04b257-7976-4309-94ad-54226bdc34f9"
+			"aa5618dc-010f-4b80-8d05-54ec1b0e4fdf" "ffba7de5-0224-4495-9d96-4e24734c3958"
+		)
+	)
