File: hardware/kicad/usb.kicad_sch (KiCad schematic)
At the start: 9 parts, among them J701 USB_C_Receptacle_USB2.0_16P, J702 USB_C_Receptacle_USB2.0_16P, J703 USB_C_Receptacle_USB2.0_16P

Commit message: layout: finish dq0 & dq1 routing
Parts:
- removed J701, J702, J703: USB_C_Receptacle_USB2.0_16P, Connector_USB:USB_C_Receptacle_GCT_USB4105-xx-A_16P_TopMnt_Horizontal, symbol Connector:USB_C_Receptacle_USB2.0_16P
- removed R701, R702, R703, R704, R705, R706: 5k1, symbol Device:R
Connections:
- no-connect marks 6 -> 0
