File: hardware/kicad/ZYNQ_PI_Zero.kicad_pcb (KiCad board)
At the start: 4 copper layers, 85.4 x 68.3 mm, 166 parts, among them J202 Conn_01x04_Pin, J203 Conn_02x03_Counter_Clockwise, J401 USB_C_Receptacle_USB2.0_16P, J501 Conn_02x20_Counter_Clockwise, J602 HDMI_A_1.4, J701 Micro_SD_Card, Q201 MMBT3904, Q601 2N7002, Q602 2N7002, Q603 2N7002, SW901 RESET, U201 xc7z007sclg225, U202 W25Q128JVS, U301 MT41K256M16TW-107_P, U401 TPS62130ARGTR, U402 TPS62130ARGTR, U403 SPX3819M5-L-3-3, U405 TPS62130ARGTR, U601 TPD4E05U06DQA, U602 TPD4E05U06DQA, U901 33.3333MHz

Commit message: pcb: improve BGA breakout
Routing:
- net /DDR/DDR_A10: track 9.94 -> 14.6 mm
- net /DDR/DDR_A13: track 11.5 -> 15.5 mm
- net /DDR/DDR_BA2: track 20.5 -> 23.8 mm
- net /DDR/DDR_A14: track 8.70 -> 11.8 mm
- net /DDR/DDR_A12: track 9.73 -> 12.7 mm
- net /DDR/DDR_~{RAS}: track 17.4 -> 20.3 mm
- net /DDR/DDR_~{CAS}: track 17.7 -> 20.6 mm
- net /DDR/DDR_A8: track 14.5 -> 17.3 mm
- net /DDR/DDR_A6: track 12.7 -> 15.4 mm
- net /DDR/DDR_A1: track 8.70 -> 11.3 mm
- net /DDR/DDR_CKE: track 6.57 -> 9.19 mm, vias 1 -> 2
- net /DDR/DDR_A5: track 18.6 -> 21.2 mm
- net /DDR/DDR_~{WE}: track 14.8 -> 17.4 mm
- net /DDR/DDR_A3: track 10.7 -> 13.2 mm, vias 2 -> 3
- net /DDR/DDR_A2: track 10.7 -> 13.2 mm
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
Commit message: feat: need switch two singals of SD inferface
Parts:
- added R306: 80R6, Resistor_SMD:R_0402_1005Metric, B.Cu at (142.5, 99.3)
- added R307: 80R6, Resistor_SMD:R_0402_1005Metric, B.Cu at (142.5, 100.1)
- C401, C402, C407, C408, C409, C411, C418, C420, C426, C431, C452, C701: footprint Capacitor_SMD:C_0805_2012Metric -> Capacitor_SMD:C_0603_1608Metric
- C419, C425, C428, C441, C444, C448, C453, C456: moved to B.Cu
- C423: footprint Capacitor_SMD:C_0805_2012Metric -> Capacitor_SMD:C_0603_1608Metric; moved to B.Cu
- F601: footprint Fuse:Fuse_0603_1608Metric -> Fuse:Fuse_0805_2012Metric
- H101, H102, H103, H104: footprint MountingHole:MountingHole_2.2mm_M2 -> MountingHole:MountingHole_3.2mm_M3
- J602: footprint Connector_Video:HDMI_A_Amphenol_10029449-x01xLF_Horizontal -> Project:HDMI-SMD_HDMI-19PIN-043_C2858275
- J701: footprint Projects:TF-SMD_503398-1892 -> Project:TF-SMD_TF-115-BCP9_LARG
- R202, R207, R401, R402, R608, R609, R901, R902, R904, R905: footprint Resistor_SMD:R_0402_1005Metric -> Resistor_SMD:R_0603_1608Metric
- R206: value 390R -> 330R; footprint Resistor_SMD:R_0402_1005Metric -> Resistor_SMD:R_0603_1608Metric
- U301: footprint Projects:BGA96C80P9X16_1400X800X120 -> Project:BGA96C80P9X16_1400X800X120
- moved Q201 117.6 mm to (111.5, 116.5), turned to 90 degrees
- moved C436 114.3 mm to (124.0, 115.2), turned to -90 degrees
- moved R202 109.3 mm to (110.0, 114.2), turned to 180 degrees
- moved R201 106.9 mm to (112.8, 113.7)
- moved R203 106.0 mm to (112.8, 112.7)
- moved D201 98.8 mm to (110.0, 112.7), turned to 180 degrees
- moved C441 95.6 mm to (143.0, 101.1)
- moved C448 92.9 mm to (146.8, 114.8), turned to -90 degrees
- moved C444 91.6 mm to (148.0, 114.8), turned to -90 degrees
- moved D902 87.6 mm to (124.8, 82.5)
- moved C453 87.5 mm to (153.2, 108.2), turned to -90 degrees
- moved C456 86.7 mm to (154.5, 108.2), turned to -90 degrees
- moved D801 85.1 mm to (135.0, 82.5)
- moved R803 82.9 mm to (135.0, 84.0), turned to 180 degrees
- moved C428 82.2 mm to (150.2, 112.8)
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Connections:
- C301 pad 2: +VTTREF -> DDR3_VREF
- C302 pad 1: +VTTREF -> DDR3_VREF
- C313 pad 1: +VTTREF -> ZYNQ_DDR_VREF
- J203 pad 2: TMS -> TDI
- J203 pad 4: TDI -> TMS
- J401 pad A6: USB_D+ -> unconnected-(J401-D+-PadA6)
- J401 pad A7: USB_D- -> unconnected-(J401-D--PadA7)
- J401 pad B6: USB_D+ -> unconnected-(J401-D+-PadB6)
- J401 pad B7: USB_D- -> unconnected-(J401-D--PadB7)
- R301 pad 1: unconnected-(R301-Pad1) -> /DDR/DDR_~{RESET}
- R304 pad 2: +VTTREF -> DDR3_VREF
- R305 pad 1: +VTTREF -> DDR3_VREF
- U201 pad F4: +VTTREF -> ZYNQ_DDR_VREF
- U201 pad G11: HDMI_HPD_N_3V3 -> unconnected-(U201B-IO_L1P_T0_34-PadG11)
- U201 pad G12: HDMI_DDC_SDA_3V3 -> unconnected-(U201B-IO_L2P_T0_34-PadG12)
- U201 pad H13: HDMI_DDC_SCL_3V3 -> unconnected-(U201B-IO_L2N_T0_34-PadH13)
- U201 pad P11: unconnected-(U201B-IO_L16P_T2_34-PadP11) -> HDMI_CLK_P
- U201 pad P8: unconnected-(U201B-IO_L23P_T3_34-PadP8) -> HDMI_DDC_SDA_3V3
- U201 pad R10: unconnected-(U201B-IO_L24N_T3_34-PadR10) -> HDMI_DDC_SCL_3V3
- U201 pad R11: unconnected-(U201B-IO_L16N_T2_34-PadR11) -> HDMI_CLK_N
- U201 pad R12: HDMI_CLK_N -> unconnected-(U201B-IO_L17P_T2_34-PadR12)
- U201 pad R13: HDMI_CLK_P -> unconnected-(U201B-IO_L17N_T2_34-PadR13)
- U201 pad R8: unconnected-(U201B-IO_L20N_T3_34-PadR8) -> HDMI_HPD_N_3V3
- U301 pad H1: +VTTREF -> DDR3_VREF
- U301 pad M8: +VTTREF -> DDR3_VREF
Routing:
- net PL_LED: track 0.00 -> 59.5 mm
- net UART_RX: track 0.00 -> 57.0 mm, vias 0 -> 1
- net /POWER/1V5_PG: track 0.00 -> 54.5 mm, vias 0 -> 3
- net UART_TX: track 0.00 -> 52.6 mm, vias 0 -> 1
- net DONE: track 0.00 -> 51.7 mm, vias 0 -> 2
- net TCK: track 0.57 -> 43.7 mm
- net /POWER/1V8_PG: track 0.00 -> 39.3 mm, vias 0 -> 3
- net /DDR/DDR_BA1: track 8.69 -> 46.9 mm
- net HDMI_HPD_N_3V3: track 0.00 -> 37.8 mm
- net +HDMI_5V: track 0.00 -> 37.6 mm, vias 0 -> 3
- net /DDR/DDR_CKE: track 9.19 -> 44.2 mm
- net /DDR/DDR_A1: track 11.3 -> 43.7 mm, vias 1 -> 2
- net /DDR/DDR_A10: track 14.6 -> 46.9 mm
- net /DDR/DDR_A14: track 11.8 -> 44.1 mm, vias 1 -> 2
- net /DDR/DDR_A11: track 11.5 -> 43.5 mm, vias 1 -> 2
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- added copper zone on B.Cu, net +1V0
- added copper zone on B.Cu, net +1V8
- added copper zone on F.Cu, net +3V3
- added copper zone on In2.Cu, net +5V
- added copper zone on B.Cu, net GND
- added copper zone on F.Cu, net GND
- added copper zone on In1.Cu, net GND
Other:
- board size 85.4 x 68.3 mm -> 79.6 x 56.2 mm
- board text added: "1V0"
- board text added: "1V5"
- board text added: "1V8"
- board text added: "3V3"
- board text added: "DONE"
- board text added: "JTAG"
- board text added: "PL LED"
- board text added: "PS LED"
- board text added: "QSPI"
- board text added: "RESET"
- board text added: "SD"
