File: hardware/kicad/bank0.kicad_sch (KiCad schematic)
At the start: 27 parts, among them J201 Conn_02x05_Odd_Even, J202 Conn_01x04_Pin, Q201 MMBT3904, U201 xc7z007sclg225, U202 W25Q256FVEI

Commit message: layout: finish dq0 & dq1 routing
Parts:
- removed J201: Conn_02x05_Odd_Even, Connector_PinSocket_2.54mm:PinSocket_2x05_P2.54mm_Vertical, symbol Connector_Generic:Conn_02x05_Odd_Even
- removed unit 4 of U201
- removed unit 3 of U201
- removed unit 7 of U201
- removed unit 5 of U201
- removed unit 2 of U201
- removed U202: W25Q256FVEI, Footprints:IC_W25N04KVZEIU, symbol W25Q256FVEI:W25Q256FVEI
- added J203: Conn_02x03_Counter_Clockwise, Connector_PinHeader_2.00mm:PinHeader_2x03_P2.00mm_Vertical, symbol Connector_Generic:Conn_02x03_Counter_Clockwise
- added U202: W25Q128JVS, Package_SO:SOIC-8_5.3x5.3mm_P1.27mm, symbol w25q128jvs:W25Q128JVS
- R207: value 470R -> 10k
Connections:
- net +1V8: now also U201.E6 (VCCBATT_0)
- net +3V3: now also U201.F6 (CFGBVS_0), U201.G4 (RSVDVCC1), U201.H4 (RSVDVCC3), U201.J4 (RSVDVCC2), U201.K8 (VCCO_0), J203.1 (Pin_1), U202.8 (VCC); no longer R208.1
- net DONE: now also U201.M7 (DONE_0)
- net GND: now also R208.1, U201.E8 (RSVDGND), U201.F8 (GNDADC_0), U201.G7 (VP_0), U201.G8 (VREFN_0), U201.H7 (VREFP_0), U201.H8 (VN_0), U201.J7 (DXP_0), J203.6 (Pin_6), U202.4 (GND)
- net INIT_B: now also U201.D5 (INIT_B_0)
- net PROGRAM_B: now also U201.K6 (PROGRAM_B_0)
- net QSPI_CLK: now also U202.6 (CLK)
- net QSPI_CS: now also U202.1 (~{CS})
- net QSPI_D0: now also U202.5 (DI/IO_{0})
- net QSPI_D1: now also U202.2 (DO/IO_{1})
- net QSPI_D2_PS_MIO4: now also U202.3 (~{WP}/IO_{2})
- net QSPI_D3_PS_MIO5: now also U202.7 (~{HOLD}/~{RESET}/IO_{3})
- net TCK: now also U201.G9 (TCK_0), J203.5 (Pin_5)
- net TDI: now also U201.L7 (TDI_0), J203.4 (Pin_4)
- net TDO: now also U201.L8 (TDO_0), J203.3 (Pin_3)
- net TMS: now also U201.L9 (TMS_0), J203.2 (Pin_2)
- net at C201.1, FB201.1: now also U201.F7 (VCCADC_0)
- no-connect marks 1 -> 0
Other:
- moved on the sheet: C201, C202, C203, FB201, R204, R205, U201A

Commit message: feat: need switch two singals of SD inferface
Parts:
- R202, R207: footprint Resistor_SMD:R_0402_1005Metric -> Resistor_SMD:R_0603_1608Metric
- R206: value 390R -> 330R; footprint Resistor_SMD:R_0402_1005Metric -> Resistor_SMD:R_0603_1608Metric
Connections:
- net TDI: now also J203.2 (Pin_2); no longer J203.4 (Pin_4)
- net TMS: now also J203.4 (Pin_4); no longer J203.2 (Pin_2)
Changed lines of the file:
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@@
 	)
 	(junction
-		(at 198.12 77.47)
-		(diameter 0)
-		(color 0 0 0 0)
-	)
-	(junction
 		(at 55.88 137.16)
 		(diameter 0)
@@
 	(wire
 		(pts
-			(xy 106.68 123.19) (xy 106.68 125.73)
-		)
-		(stroke
-			(width 0)
-			(type default)
-		)
-	)
-	(wire
-		(pts
 			(xy 49.53 137.16) (xy 55.88 137.16)
 		)
@@
 	(wire
 		(pts
-			(xy 93.98 123.19) (xy 93.98 125.73)
-		)
-		(stroke
-			(width 0)
-			(type default)
-		)
-	)
-	(wire
-		(pts
 			(xy 99.06 57.15) (xy 49.53 57.15)
 		)
@@
 	(wire
 		(pts
-			(xy 198.12 77.47) (xy 198.12 78.74)
+			(xy 198.12 74.93) (xy 198.12 78.74)
 		)
 		(stroke
@@
 	(wire
 		(pts
-			(xy 198.12 77.47) (xy 196.85 77.47)
-		)
-		(stroke
-			(width 0)
-			(type default)
-		)
-	)
-	(wire
-		(pts
 			(xy 35.56 167.64) (xy 39.37 167.64)
 		)
@@
 	(wire
 		(pts
-			(xy 198.12 74.93) (xy 198.12 77.47)
-		)
-		(stroke
-			(width 0)
-			(type default)
-		)
-	)
-	(wire
-		(pts
 			(xy 49.53 52.07) (xy 64.77 52.07)
 		)
@@
 	(wire
 		(pts
-			(xy 93.98 125.73) (xy 106.68 125.73)
-		)
-		(stroke
-			(width 0)
-			(type default)
-		)
-	)
-	(wire
-		(pts
 			(xy 88.9 101.6) (xy 88.9 95.25)
 		)
@@
 	(global_label "TDI"
 		(shape input)
-		(at 116.84 161.29 0)
+		(at 99.06 158.75 180)
 		(effects
 			(font
 				(size 1.27 1.27)
 			)
-			(justify left)
+			(justify right)
 		)
 		(property "Intersheetrefs" "${INTERSHEET_REFS}"
-			(at 116.84 161.29 0)
+			(at 99.06 158.75 0)
 			(hide yes)
 			(show_name no)
@@
 	(global_label "TMS"
 		(shape input)
-		(at 99.06 158.75 180)
+		(at 116.84 161.29 0)
 		(effects
 			(font
 				(size 1.27 1.27)
 			)
-			(justify right)
+			(justify left)
 		)
 		(property "Intersheetrefs" "${INTERSHEET_REFS}"
-			(at 99.06 158.75 0)
+			(at 116.84 161.29 0)
 			(hide yes)
 			(show_name no)
@@
 	)
 	(symbol
-		(lib_id "power:+FPGA_VREF")
-		(at 97.79 152.4 0)
-		(unit 1)
-		(body_style 1)
-		(exclude_from_sim no)
-		(in_bom yes)
-		(on_board yes)
-		(in_pos_files yes)
-		(dnp no)
-		(property "Reference" "#PWR0231"
-			(at 97.79 156.21 0)
-			(hide yes)
-			(show_name no)
-			(do_not_autoplace no)
-			(effects
-				(font
-					(size 1.27 1.27)
-				)
-			)
-		)
-		(property "Value" "+FPGA_VREF"
-			(at 97.79 148.59 0)
-			(show_name no)
-			(do_not_autoplace no)
-			(effects
-				(font
-					(size 1.27 1.27)
-				)
-			)
-		)
-		(property "Footprint" ""
-			(at 97.79 152.4 0)
-			(hide yes)
-			(show_name no)
-			(do_not_autoplace no)
-			(effects
-				(font
-					(size 1.27 1.27)
-				)
-			)
-		)
-		(property "Datasheet" ""
-			(at 97.79 152.4 0)
-			(hide yes)
-			(show_name no)
-			(do_not_autoplace no)
-			(effects
-				(font
-					(size 1.27 1.27)
-				)
-			)
-		)
-		(property "Description" "Power symbol creates a global label with name \"+FPGA_VREF\""
-			(at 97.79 152.4 0)
-			(hide yes)
-			(show_name no)
-			(do_not_autoplace no)
-			(effects
-				(font
-					(size 1.27 1.27)
-				)
-			)
-		)
-		(pin "1"
-		)
-		(instances
-			(project "ZYNQ_PI_Zero"
-				(path "/e0cc3273-981b-466d-ad17-67861c989a34/13f5c536-9334-4878-b77d-62113dbf22d4"
-					(reference "#PWR0231")
-					(unit 1)
-				)
-			)
-		)
-	)
-	(symbol
 		(lib_id "power:GND")
 		(at 173.99 88.9 0)
@@
 	(symbol
 		(lib_id "power:+3V3")
-		(at 106.68 123.19 0)
+		(at 97.79 152.4 0)
 		(unit 1)
 		(body_style 1)
@@
 		(in_pos_files yes)
 		(dnp no)
-		(property "Reference" "#PWR0215"
-			(at 106.68 127 0)
+		(property "Reference" "#PWR0214"
+			(at 97.79 156.21 0)
 			(hide yes)
 			(show_name no)
@@
 		)
 		(property "Value" "+3V3"
-			(at 106.68 119.38 0)
+			(at 97.79 148.59 0)
 			(show_name no)
 			(do_not_autoplace no)
@@
 		)
 		(property "Footprint" ""
-			(at 106.68 123.19 0)
+			(at 97.79 152.4 0)
 			(hide yes)
 			(show_name no)
@@
 		)
 		(property "Datasheet" ""
-			(at 106.68 123.19 0)
+			(at 97.79 152.4 0)
 			(hide yes)
 			(show_name no)
@@
 		)
 		(property "Description" "Power symbol creates a global label with name \"+3V3\""
-			(at 106.68 123.19 0)
+			(at 97.79 152.4 0)
 			(hide yes)
 			(show_name no)
@@
 			(project "ZYNQ_PI_Zero"
 				(path "/e0cc3273-981b-466d-ad17-67861c989a34/13f5c536-9334-4878-b77d-62113dbf22d4"
-					(reference "#PWR0215")
+					(reference "#PWR0214")
 					(unit 1)
 				)
@@
 			)
 		)
-		(property "Value" "390R"
+		(property "Value" "330R"
 			(at 176.53 83.8199 0)
 			(show_name no)
@@
 			)
 		)
-		(property "Footprint" "Resistor_SMD:R_0402_1005Metric"
+		(property "Footprint" "Resistor_SMD:R_0603_1608Metric"
 			(at 172.212 82.55 90)
 			(hide yes)
@@
 			)
 		)
-		(property "Footprint" "Resistor_SMD:R_0402_1005Metric"
+		(property "Footprint" "Resistor_SMD:R_0603_1608Metric"
 			(at 186.182 113.03 90)
 			(hide yes)
@@
 	)
 	(symbol
-		(lib_id "power:+FPGA_VREF")
-		(at 93.98 123.19 0)
-		(unit 1)
-		(body_style 1)
-		(exclude_from_sim no)
-		(in_bom yes)
-		(on_board yes)
-		(in_pos_files yes)
-		(dnp no)
-		(property "Reference" "#PWR0214"
-			(at 93.98 127 0)
-			(hide yes)
-			(show_name no)
-			(do_not_autoplace no)
-			(effects
-				(font
-					(size 1.27 1.27)
-				)
-			)
-		)
-		(property "Value" "+FPGA_VREF"
-			(at 93.98 119.38 0)
-			(show_name no)
-			(do_not_autoplace no)
-			(effects
-				(font
-					(size 1.27 1.27)
-				)
-			)
-		)
-		(property "Footprint" ""
-			(at 93.98 123.19 0)
-			(hide yes)
-			(show_name no)
-			(do_not_autoplace no)
-			(effects
-				(font
-					(size 1.27 1.27)
-				)
-			)
-		)
-		(property "Datasheet" ""
-			(at 93.98 123.19 0)
-			(hide yes)
-			(show_name no)
-			(do_not_autoplace no)
-			(effects
-				(font
-					(size 1.27 1.27)
-				)
-			)
-		)
-		(property "Description" "Power symbol creates a global label with name \"+FPGA_VREF\""
-			(at 93.98 123.19 0)
-			(hide yes)
-			(show_name no)
-			(do_not_autoplace no)
-			(effects
-				(font
-					(size 1.27 1.27)
-				)
-			)
-		)
-		(pin "1"
-		)
-		(instances
-			(project "ZYNQ_PI_Zero"
-				(path "/e0cc3273-981b-466d-ad17-67861c989a34/13f5c536-9334-4878-b77d-62113dbf22d4"
-					(reference "#PWR0214")
-					(unit 1)
-				)
-			)
-		)
-	)
-	(symbol
 		(lib_id "power:GND")
 		(at 231.14 50.8 0)
@@
 			)
 		)
-		(property "Footprint" "Resistor_SMD:R_0402_1005Metric"
+		(property "Footprint" "Resistor_SMD:R_0603_1608Metric"
 			(at 54.102 130.81 90)
 			(hide yes)
