File: hardware/kicad/io.kicad_sch (KiCad schematic)
At the start: 6 parts, among them SW801 PL_KEY, U201 xc7z007sclg225

Commit message: finish basic ddr routing
Parts:
- removed R801: 10k, Resistor_SMD:R_0402_1005Metric, symbol Device:R
- removed R802: 100R, Resistor_SMD:R_0402_1005Metric, symbol Device:R
- removed SW801: PL_KEY, Button_Switch_SMD:SW_Tactile_SPST_NO_Straight_CK_PTS636Sx25SMTRLFS, symbol Switch:SW_Push
Connections:
- net PL_KEY is gone; now on net HDMI_D2_P: U201.J15 (IO_L4P_T0_34)
- net HDMI_CLK_N: now also U201.R12 (IO_L17P_T2_34); no longer U201.E13 (IO_L1N_T0_AD0N_35)
- net HDMI_CLK_P: now also U201.R13 (IO_L17N_T2_34); no longer U201.F12 (IO_L1P_T0_AD0P_35)
- net HDMI_D0_N: now also U201.R15 (IO_L15N_T2_DQS_34); no longer U201.E12 (IO_L2N_T0_AD8N_35)
- net HDMI_D0_P: now also U201.P15 (IO_L15P_T2_DQS_34); no longer U201.E11 (IO_L2P_T0_AD8P_35)
- net HDMI_D1_N: now also U201.M15 (IO_L8N_T1_34); no longer U201.F14 (IO_L3N_T0_DQS_AD1N_35)
- net HDMI_D1_P: now also U201.L15 (IO_L8P_T1_34); no longer U201.F13 (IO_L3P_T0_DQS_AD1P_35)
- net HDMI_D2_N: now also U201.K15 (IO_L4N_T0_34); no longer U201.F15 (IO_L5N_T0_AD9N_35)
- net HDMI_D2_P: no longer U201.G15 (IO_L5P_T0_AD9P_35)
- net PL_LED: now also U201.G14 (IO_L3P_T0_DQS_PUDC_B_34); no longer U201.J14 (IO_L5N_T0_34)
- no-connect marks 41 -> 33

Commit message: feat: need switch two singals of SD inferface
Parts:
- U201: footprint Package_BGA:Xilinx_CLG225 -> (none)
Connections:
- net HDMI_CLK_N: now also U201.R11 (IO_L16N_T2_34); no longer U201.R12 (IO_L17P_T2_34)
- net HDMI_CLK_P: now also U201.P11 (IO_L16P_T2_34); no longer U201.R13 (IO_L17N_T2_34)
- net HDMI_DDC_SCL_3V3: now also U201.R10 (IO_L24N_T3_34); no longer U201.H13 (IO_L2N_T0_34)
- net HDMI_DDC_SDA_3V3: now also U201.P8 (IO_L23P_T3_34); no longer U201.G12 (IO_L2P_T0_34)
- net HDMI_HPD_N_3V3: now also U201.R8 (IO_L20N_T3_34); no longer U201.G11 (IO_L1P_T0_34)
- no-connect marks 33 -> 42
Changed lines of the file:
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@@
+	)
+	(no_connect
+		(at 196.85 48.26)
+	)
+	(no_connect
+		(at 196.85 63.5)
 	)
 	(no_connect
@@
 	)
 	(no_connect
+		(at 196.85 45.72)
+	)
+	(no_connect
 		(at 80.01 96.52)
 	)
@@
 	)
 	(no_connect
-		(at 80.01 157.48)
-	)
-	(no_connect
 		(at 80.01 139.7)
 	)
@@
 	)
 	(no_connect
+		(at 80.01 124.46)
+	)
+	(no_connect
+		(at 196.85 53.34)
+	)
+	(no_connect
 		(at 80.01 109.22)
 	)
@@
 	)
 	(no_connect
+		(at 196.85 58.42)
+	)
+	(no_connect
+		(at 80.01 53.34)
+	)
+	(no_connect
 		(at 80.01 147.32)
 	)
@@
 	)
 	(no_connect
+		(at 80.01 121.92)
+	)
+	(no_connect
 		(at 80.01 78.74)
 	)
@@
 	)
 	(no_connect
-		(at 80.01 119.38)
-	)
-	(no_connect
-		(at 80.01 116.84)
-	)
-	(no_connect
 		(at 80.01 76.2)
 	)
@@
 	)
 	(no_connect
-		(at 80.01 137.16)
+		(at 80.01 48.26)
 	)
 	(no_connect
@@
 	)
 	(no_connect
+		(at 80.01 50.8)
+	)
+	(no_connect
 		(at 80.01 132.08)
 	)
 	(no_connect
-		(at 80.01 154.94)
+		(at 196.85 55.88)
+	)
+	(no_connect
+		(at 196.85 60.96)
 	)
 	(no_connect
@@
 	)
 	(no_connect
+		(at 196.85 50.8)
+	)
+	(no_connect
 		(at 80.01 86.36)
+	)
+	(no_connect
+		(at 80.01 55.88)
 	)
 	(no_connect
@@
 	(wire
 		(pts
-			(xy 63.5 160.02) (xy 63.5 162.56)
+			(xy 55.88 160.02) (xy 55.88 162.56)
 		)
 		(stroke
@@
 	(wire
 		(pts
-			(xy 63.5 162.56) (xy 80.01 162.56)
+			(xy 55.88 162.56) (xy 80.01 162.56)
 		)
 		(stroke
@@
 		)
 	)
-	(global_label "HDMI_DDC_SCL_3V3"
+	(global_label "HDMI_D0_P"
 		(shape input)
-		(at 80.01 50.8 180)
+		(at 80.01 114.3 180)
 		(fields_autoplaced yes)
 		(effects
@@
 		)
 		(property "Intersheetrefs" "${INTERSHEET_REFS}"
-			(at 58.6401 50.8 0)
+			(at 66.6834 114.3 0)
 			(hide yes)
 			(show_name no)
@@
 		)
 	)
-	(global_label "HDMI_D0_P"
+	(global_label "HDMI_CLK_P"
 		(shape input)
-		(at 80.01 114.3 180)
+		(at 80.01 119.38 180)
 		(fields_autoplaced yes)
 		(effects
@@
 		)
 		(property "Intersheetrefs" "${INTERSHEET_REFS}"
-			(at 66.6834 114.3 0)
+			(at 65.5948 119.38 0)
 			(hide yes)
 			(show_name no)
@@
 		)
 	)
-	(global_label "HDMI_CLK_P"
+	(global_label "HDMI_DDC_SCL_3V3"
 		(shape input)
-		(at 80.01 121.92 180)
+		(at 80.01 157.48 180)
 		(fields_autoplaced yes)
 		(effects
@@
 		)
 		(property "Intersheetrefs" "${INTERSHEET_REFS}"
-			(at 65.5948 121.92 0)
+			(at 58.6401 157.48 0)
+			(hide yes)
+			(show_name no)
+			(do_not_autoplace no)
+			(effects
+				(font
+					(size 1.27 1.27)
+				)
+				(justify right)
+			)
+		)
+	)
+	(global_label "HDMI_HPD_N_3V3"
+		(shape input)
+		(at 80.01 137.16 180)
+		(fields_autoplaced yes)
+		(effects
+			(font
+				(size 1.27 1.27)
+			)
+			(justify right)
+		)
+		(property "Intersheetrefs" "${INTERSHEET_REFS}"
+			(at 60.7567 137.16 0)
 			(hide yes)
 			(show_name no)
@@
 		)
 	)
+	(global_label "HDMI_CLK_N"
+		(shape input)
+		(at 80.01 116.84 180)
+		(fields_autoplaced yes)
+		(effects
+			(font
+				(size 1.27 1.27)
+			)
+			(justify right)
+		)
+		(property "Intersheetrefs" "${INTERSHEET_REFS}"
+			(at 65.5343 116.84 0)
+			(hide yes)
+			(show_name no)
+			(do_not_autoplace no)
+			(effects
+				(font
+					(size 1.27 1.27)
+				)
+				(justify right)
+			)
+		)
+	)
 	(global_label "HDMI_D0_N"
 		(shape input)
@@
 		)
 	)
-	(global_label "HDMI_CLK_N"
+	(global_label "HDMI_DDC_SDA_3V3"
 		(shape input)
-		(at 80.01 124.46 180)
+		(at 80.01 154.94 180)
 		(fields_autoplaced yes)
 		(effects
@@
 		)
 		(property "Intersheetrefs" "${INTERSHEET_REFS}"
-			(at 65.5343 124.46 0)
+			(at 58.5796 154.94 0)
 			(hide yes)
 			(show_name no)
@@
 		)
 	)
-	(global_label "HDMI_HPD_N_3V3"
+	(global_label "PL_LED"
 		(shape input)
-		(at 80.01 48.26 180)
+		(at 248.92 147.32 0)
 		(fields_autoplaced yes)
 		(effects
@@
 				(size 1.27 1.27)
 			)
-			(justify right)
+			(justify left)
 		)
 		(property "Intersheetrefs" "${INTERSHEET_REFS}"
-			(at 60.7567 48.26 0)
-			(hide yes)
-			(show_name no)
-			(do_not_autoplace no)
-			(effects
-				(font
-					(size 1.27 1.27)
-				)
-				(justify right)
-			)
-		)
-	)
-	(global_label "HDMI_DDC_SDA_3V3"
+			(at 258.618 147.32 0)
+			(hide yes)
+			(show_name no)
+			(do_not_autoplace no)
+			(effects
+				(font
+					(size 1.27 1.27)
+				)
+				(justify left)
+			)
+		)
+	)
+	(global_label "PL_LED"
 		(shape input)
-		(at 80.01 53.34 180)
+		(at 80.01 58.42 180)
 		(fields_autoplaced yes)
 		(effects
@@
 		)
 		(property "Intersheetrefs" "${INTERSHEET_REFS}"
-			(at 58.5796 53.34 0)
-			(hide yes)
-			(show_name no)
-			(do_not_autoplace no)
-			(effects
-				(font
-					(size 1.27 1.27)
-				)
-				(justify right)
-			)
-		)
-	)
-	(global_label "PL_LED"
-		(shape input)
-		(at 248.92 147.32 0)
-		(fields_autoplaced yes)
-		(effects
-			(font
-				(size 1.27 1.27)
-			)
-			(justify left)
-		)
-		(property "Intersheetrefs" "${INTERSHEET_REFS}"
-			(at 258.618 147.32 0)
-			(hide yes)
-			(show_name no)
-			(do_not_autoplace no)
-			(effects
-				(font
-					(size 1.27 1.27)
-				)
-				(justify left)
-			)
-		)
-	)
-	(global_label "PL_LED"
-		(shape input)
-		(at 80.01 58.42 180)
-		(fields_autoplaced yes)
-		(effects
-			(font
-				(size 1.27 1.27)
-			)
-			(justify right)
-		)
-		(property "Intersheetrefs" "${INTERSHEET_REFS}"
 			(at 70.312 58.42 0)
 			(hide yes)
@@
 	(symbol
 		(lib_id "power:+3V3")
-		(at 63.5 160.02 0)
+		(at 55.88 160.02 0)
 		(unit 1)
 		(body_style 1)
@@
 		(dnp no)
 		(property "Reference" "#PWR0801"
-			(at 63.5 163.83 0)
+			(at 55.88 163.83 0)
 			(hide yes)
 			(show_name no)
@@
 		)
 		(property "Value" "+3V3"
-			(at 63.5 156.21 0)
+			(at 55.88 156.21 0)
 			(show_name no)
 			(do_not_autoplace no)
@@
 		)
 		(property "Footprint" ""
-			(at 63.5 160.02 0)
+			(at 55.88 160.02 0)
 			(hide yes)
 			(show_name no)
@@
 		)
 		(property "Datasheet" ""
-			(at 63.5 160.02 0)
+			(at 55.88 160.02 0)
 			(hide yes)
 			(show_name no)
@@
 		)
 		(property "Description" "Power symbol creates a global label with name \"+3V3\""
-			(at 63.5 160.02 0)
+			(at 55.88 160.02 0)
 			(hide yes)
 			(show_name no)
@@
 	)
 	(symbol
+		(lib_name "xc7z007sclg225_1")
 		(lib_id "Xilinx7:xc7z007sclg225")
 		(at 80.01 45.72 0)
@@
 			)
 		)
-		(property "Footprint" "Package_BGA:Xilinx_CLG225"
+		(property "Footprint" ""
 			(at 85.09 44.45 0)
 			(hide yes)
@@
 			)
 		)
-		(property "Footprint" "Package_BGA:Xilinx_CLG225"
+		(property "Footprint" ""
 			(at 201.93 44.45 0)
 			(hide yes)
